File: hardware/KiCad/UVK5_Reversing20230702_kicad 2/RX_path_sch.kicad_sch (KiCad schematic)
At the start: 42 parts, among them J201 Conn_Coaxial, J202 Conn_Coaxial, J203 Conn_Coaxial, Q201 2SC3356, Q202 2SC3356

Commit message: 27-08-2023
Parts:
- C21: renamed from C201; symbol Device:C_Small -> UV-K5:C_Small
- C22: renamed from C203; symbol Device:C_Small -> UV-K5:C_Small
- C23: renamed from C204; symbol Device:C_Small -> UV-K5:C_Small
- C24: renamed from C205; symbol Device:C_Small -> UV-K5:C_Small
- C25: renamed from C208; symbol Device:C_Small -> UV-K5:C_Small
- C26: renamed from C207; symbol Device:C_Small -> UV-K5:C_Small
- C27: renamed from C209; symbol Device:C_Small -> UV-K5:C_Small
- C28: renamed from C210; symbol Device:C_Small -> UV-K5:C_Small
- C29: renamed from C211; symbol Device:C_Small -> UV-K5:C_Small
- C30: renamed from C212; symbol Device:C_Small -> UV-K5:C_Small
- C31: renamed from C213; symbol Device:C_Small -> UV-K5:C_Small
- C32: renamed from C215; symbol Device:C_Small -> UV-K5:C_Small
- C33: renamed from C216; symbol Device:C_Small -> UV-K5:C_Small
- C34: renamed from C219; symbol Device:C_Small -> UV-K5:C_Small
- C35: renamed from C220; symbol Device:C_Small -> UV-K5:C_Small
- C36: renamed from C221; symbol Device:C_Small -> UV-K5:C_Small
- D21: renamed from D201; symbol Device:D -> UV-K5:D
- D22: renamed from D202; symbol Device:D -> UV-K5:D
- D23: renamed from D203; symbol Device:D -> UV-K5:D
- D24: renamed from D204; symbol Device:D -> UV-K5:D
- J21: renamed from J201; symbol Connector:Conn_Coaxial -> UV-K5:Conn_Coaxial
- J22: renamed from J202; symbol Connector:Conn_Coaxial -> UV-K5:Conn_Coaxial
- J23: renamed from J203; symbol Connector:Conn_Coaxial -> UV-K5:Conn_Coaxial
- L21: renamed from L201; symbol Device:L -> UV-K5:L
- L22: renamed from L202; symbol Device:L -> UV-K5:L
- L23: renamed from L204; symbol Device:L -> UV-K5:L
- L24: renamed from L203; symbol Device:L -> UV-K5:L
- L25: renamed from L205; symbol Device:L -> UV-K5:L
- L26: renamed from L206; symbol Device:L -> UV-K5:L
- L27: renamed from L208; symbol Device:L -> UV-K5:L
- Q21: renamed from Q201; symbol Transistor_BJT:BFR92 -> UV-K5:BFR92
- Q22: renamed from Q202; symbol Transistor_BJT:BFR92 -> UV-K5:BFR92
- R21: renamed from R201; symbol Device:R -> UV-K5:R
- R22: renamed from R202; symbol Device:R -> UV-K5:R
- R23: renamed from R203; symbol Device:R -> UV-K5:R
- R24: renamed from R204; symbol Device:R -> UV-K5:R
- R25: renamed from R205; symbol Device:R -> UV-K5:R
- R26: renamed from R206; symbol Device:R -> UV-K5:R
- R27: renamed from R207; symbol Device:R -> UV-K5:R
- R28: renamed from R208; symbol Device:R -> UV-K5:R
- R29: renamed from R210; symbol Device:R -> UV-K5:R
- R30: renamed from R209; symbol Device:R -> UV-K5:R
