File: hardware/KiCad/UVK5_Reversing20230702_kicad 2/TX_chain_sch.kicad_sch (KiCad schematic)
At the start: 109 parts, among them J301 ANT, Q1 2SC3356, Q2 2SK3078, Q3 RD02LUS2, Q301 DTC114E, Q302 DTC114E

Commit message: 27-08-2023
Parts:
- removed C339: 470pF, symbol Device:C_Small
- removed L323: 1uH, symbol Device:L
- added L47: L, symbol UV-K5:L
- C110: renamed from C318; value 15pF -> C_Small; symbol Device:C_Small -> UV-K5:C_Small
- C162: renamed from C323; value 16pF -> C_Small; symbol Device:C_Small -> UV-K5:C_Small
- C37: renamed from C301; symbol Device:C_Small -> UV-K5:C_Small
- C38: renamed from C302; symbol Device:C_Small -> UV-K5:C_Small
- C39: renamed from C303; symbol Device:C_Small -> UV-K5:C_Small
- C40: renamed from C304; symbol Device:C_Small -> UV-K5:C_Small
- C41: renamed from C305; symbol Device:C_Small -> UV-K5:C_Small
- C42: renamed from C312; symbol Device:C_Small -> UV-K5:C_Small
- C43: renamed from C306; symbol Device:C_Small -> UV-K5:C_Small
- C44: renamed from C309; symbol Device:C_Small -> UV-K5:C_Small
- C45: renamed from C322; symbol Device:C_Small -> UV-K5:C_Small
- C46: renamed from C316; symbol Device:C_Small -> UV-K5:C_Small
- C47: renamed from C307; symbol Device:C_Small -> UV-K5:C_Small
- C48: renamed from C317; symbol Device:C_Small -> UV-K5:C_Small
- C49: renamed from C319; symbol Device:C_Small -> UV-K5:C_Small
- C50: renamed from C320; symbol Device:C_Small -> UV-K5:C_Small
- C51: renamed from C321; symbol Device:C_Small -> UV-K5:C_Small
- C52: renamed from C308; symbol Device:C_Small -> UV-K5:C_Small
- C53: renamed from C310; symbol Device:C_Small -> UV-K5:C_Small
- C54: renamed from C311; symbol Device:C_Small -> UV-K5:C_Small
- C55: renamed from C315; symbol Device:C_Small -> UV-K5:C_Small
- C56: renamed from C313; symbol Device:C_Small -> UV-K5:C_Small
- C57: renamed from C324; symbol Device:C_Small -> UV-K5:C_Small
- C58: renamed from C328; symbol Device:C_Small -> UV-K5:C_Small
- C59: renamed from C325; symbol Device:C_Small -> UV-K5:C_Small
- C60: renamed from C326; symbol Device:C_Small -> UV-K5:C_Small
- C61: renamed from C338; symbol Device:C_Small -> UV-K5:C_Small
- C62: renamed from C327; symbol Device:C_Small -> UV-K5:C_Small
- C63: renamed from C329; symbol Device:C_Small -> UV-K5:C_Small
- C64: renamed from C330; symbol Device:C_Small -> UV-K5:C_Small
- C65: renamed from C331; symbol Device:C_Small -> UV-K5:C_Small
- C66: renamed from C314; symbol Device:C_Small -> UV-K5:C_Small
- C67: renamed from C332; symbol Device:C_Small -> UV-K5:C_Small
- C69: renamed from C21; symbol Device:C_Small -> UV-K5:C_Small
- C70: renamed from C334; symbol Device:C_Small -> UV-K5:C_Small
- C71: renamed from C335; symbol Device:C_Small -> UV-K5:C_Small
- C72: renamed from C336; symbol Device:C_Small -> UV-K5:C_Small
- C74: renamed from C333; symbol Device:C_Small -> UV-K5:C_Small
- C75: renamed from C337; symbol Device:C_Small -> UV-K5:C_Small
- C76: renamed from C339; symbol Device:C_Small -> UV-K5:C_Small
- C77: renamed from C341; symbol Device:C_Small -> UV-K5:C_Small
- C78: renamed from C342; symbol Device:C_Small -> UV-K5:C_Small
- C79: renamed from C343; symbol Device:C_Small -> UV-K5:C_Small
- C80: renamed from C344; symbol Device:C_Small -> UV-K5:C_Small
- C81: renamed from C345; symbol Device:C_Small -> UV-K5:C_Small
- C82: renamed from C340; symbol Device:C_Small -> UV-K5:C_Small
- C83: renamed from C346; symbol Device:C_Small -> UV-K5:C_Small
- C84: renamed from C347; symbol Device:C_Small -> UV-K5:C_Small
- C85: renamed from C348; symbol Device:C_Small -> UV-K5:C_Small
- D25: renamed from D304; symbol Device:D -> UV-K5:D
- D26: renamed from D303; symbol Device:D -> UV-K5:D
- D27: renamed from D301; symbol Device:D -> UV-K5:D
- D28: renamed from D302; symbol Device:D -> UV-K5:D
- D29: renamed from D305; symbol Device:D -> UV-K5:D
- D30: renamed from D306; symbol Device:D -> UV-K5:D
- D31: renamed from D307; symbol Device:D -> UV-K5:D
- D32: renamed from D308; symbol Device:D -> UV-K5:D
- D33: renamed from D309; symbol Device:D -> UV-K5:D
- D34: renamed from D310; symbol Device:D -> UV-K5:D
- D35: renamed from D311; symbol Device:D -> UV-K5:D
- D36: renamed from D312; symbol Device:D -> UV-K5:D
- J24: renamed from J301; symbol Connector:Conn_Coaxial -> UV-K5:Conn_Coaxial
- L28: renamed from L312; symbol Device:L -> UV-K5:L
- L29: renamed from L302; symbol Device:L -> UV-K5:L
- L30: renamed from L306; symbol Device:L -> UV-K5:L
- L31: renamed from L301; symbol Device:L -> UV-K5:L
- L32: renamed from L307; symbol Device:L -> UV-K5:L
- L33: renamed from L313; symbol Device:L -> UV-K5:L
- L34: renamed from L309; symbol Device:L -> UV-K5:L
- L35: renamed from L310; symbol Device:L -> UV-K5:L
- L36: renamed from L311; symbol Device:L -> UV-K5:L
- L37: renamed from L303; value 1uH? -> RFC; symbol Device:L -> UV-K5:L
- L38: renamed from L304; value 100nH -> L; symbol Device:L -> UV-K5:L
- L39: renamed from L305; value 20nH -> L; symbol Device:L -> UV-K5:L
- L40: renamed from L315; symbol Device:L -> UV-K5:L
- L41: renamed from L308; symbol Device:L -> UV-K5:L
- L42: renamed from L317; symbol Device:L -> UV-K5:L
- L43: renamed from L318; symbol Device:L -> UV-K5:L
- L44: renamed from L319; symbol Device:L -> UV-K5:L
- L45: renamed from L320; symbol Device:L -> UV-K5:L
- L46: renamed from L322; symbol Device:L -> UV-K5:L
- L48: renamed from L321; symbol Device:L -> UV-K5:L
- L49: renamed from L324; symbol Device:L -> UV-K5:L
- L50: renamed from L325; symbol Device:L -> UV-K5:L
- L51: renamed from L326; symbol Device:L -> UV-K5:L
- L52: renamed from L327; symbol Device:L -> UV-K5:L
- L53: renamed from L328; symbol Device:L -> UV-K5:L
- L54: renamed from L329; symbol Device:L -> UV-K5:L
- Q01: renamed from Q1; value 2SC3356 -> 2SC3356,R24; symbol Transistor_BJT:BFR92 -> UV-K5:BFR92
- Q02: renamed from Q2; value 2SK3078 -> 2SK3078,UW; symbol Transistor_FET:IRF540N -> UV-K5:IRF540N
- Q03: renamed from Q301; symbol Transistor_BJT:DTC114E -> UV-K5:DTC114E
- Q24: renamed from Q302; symbol Transistor_BJT:DTC114E -> UV-K5:DTC114E
- Q27: renamed from Q3; symbol Transistor_FET:IRF540N -> UV-K5:IRF540N
- R31: renamed from R301; symbol Device:R -> UV-K5:R
- R32: renamed from R302; symbol Device:R -> UV-K5:R
- R33: renamed from R303; symbol Device:R -> UV-K5:R
- R34: renamed from R306; symbol Device:R -> UV-K5:R
- R35: renamed from R307; symbol Device:R -> UV-K5:R
- R36: renamed from R304; value 10 -> R; symbol Device:R -> UV-K5:R
- R37: renamed from R305; value 220 -> R; symbol Device:R -> UV-K5:R
- R38: renamed from R308; symbol Device:R -> UV-K5:R
- R39: renamed from R310; symbol Device:R -> UV-K5:R
- R40: renamed from R309; value 33k -> R; symbol Device:R -> UV-K5:R
- R41: renamed from R311; symbol Device:R -> UV-K5:R
- R42: renamed from R312; symbol Device:R -> UV-K5:R
- R43: renamed from R313; symbol Device:R -> UV-K5:R
- R44: renamed from R314; symbol Device:R -> UV-K5:R
Connections:
- net VIA_204: now also L47.2
- net at C61.1, C62.2, L40.1: no longer D32.1 (K)
- net at J24.1 (In), L40.2: now also D32.1 (K), L47.1
- net BK4819_TX renamed BK4819_Pout
Other:
- moved on the sheet: C162, C37, C39, C40, C41, C42, C43, C44, C45, C46, C48, C49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
