File: hardware/KiCad/Kicad_UVK5_reversing20230909/Keypad.kicad_sch (KiCad schematic)
At the start: 36 parts, among them SW21 M / A (10), SW22 1, SW23 4, SW24 7, SW25 UP / B (11), SW26 2, SW27 5, SW28 8, SW29 DOWN / C (12), SW30 3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

Commit message: Add files via upload
Parts:
- added R193, R206: 100R, symbol UV-K5:R
- added R223, R227: 1k, symbol UV-K5:R
Connections:
- net PA3: now also R227.1; no longer R62.2, R72.2, SW21.2, SW25.2, SW29.2, SW33.2, SW37.1
- net PA4: now also R223.1; no longer R63.2, R73.2, SW22.2, SW26.2, SW30.2, SW34.2, SW38.1
- net PA5: now also R206.1; no longer R64.2, SW23.2, SW27.2, SW31.2, SW35.2
- net PA6: now also R193.1; no longer R65.2, SW24.2, SW28.2, SW32.2, SW36.2
- net PC5: no longer R69.2, SW39.1
- new net: R227.2, R62.2, R72.2, SW21.2, SW25.2, SW29.2, SW33.2, SW37.1
- new net: R223.2, R63.2, R73.2, SW22.2, SW26.2, SW30.2, SW34.2, SW38.1
- new net: R193.2, R65.2, SW24.2, SW28.2, SW32.2, SW36.2
- new net: R206.2, R64.2, SW23.2, SW27.2, SW31.2, SW35.2
- new net: R69.2, SW39.1
Other:
- note added: "√"
Changed lines of the file:
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@@
     (stroke (width 0) (type default))
   )
-  (wire (pts (xy 35.56 101.6) (xy 100.33 101.6))
+  (wire (pts (xy 35.56 101.6) (xy 39.37 101.6))
     (stroke (width 0) (type default))
   )
@@
     (stroke (width 0) (type default))
   )
+  (wire (pts (xy 46.99 91.44) (xy 59.69 91.44))
+    (stroke (width 0) (type default))
+  )
   (wire (pts (xy 93.98 25.4) (xy 93.98 40.64))
     (stroke (width 0) (type default))
@@
     (stroke (width 0) (type default))
   )
-  (wire (pts (xy 35.56 91.44) (xy 59.69 91.44))
+  (wire (pts (xy 35.56 91.44) (xy 39.37 91.44))
     (stroke (width 0) (type default))
   )
@@
     (stroke (width 0) (type default))
   )
+  (wire (pts (xy 46.99 93.98) (xy 77.47 93.98))
+    (stroke (width 0) (type default))
+  )
   (wire (pts (xy 67.31 25.4) (xy 67.31 27.94))
     (stroke (width 0) (type default))
@@
     (stroke (width 0) (type default))
   )
+  (wire (pts (xy 46.99 96.52) (xy 93.98 96.52))
+    (stroke (width 0) (type default))
+  )
   (wire (pts (xy 69.85 111.76) (xy 69.85 114.3))
     (stroke (width 0) (type default))
@@
     (stroke (width 0) (type default))
   )
-  (wire (pts (xy 35.56 93.98) (xy 77.47 93.98))
+  (wire (pts (xy 35.56 93.98) (xy 39.37 93.98))
     (stroke (width 0) (type default))
   )
@@
     (stroke (width 0) (type default))
   )
+  (wire (pts (xy 46.99 99.06) (xy 110.49 99.06))
+    (stroke (width 0) (type default))
+  )
   (wire (pts (xy 59.69 111.76) (xy 59.69 114.3))
     (stroke (width 0) (type default))
@@
     (stroke (width 0) (type default))
   )
-  (wire (pts (xy 35.56 96.52) (xy 93.98 96.52))
+  (wire (pts (xy 35.56 96.52) (xy 39.37 96.52))
     (stroke (width 0) (type default))
   )
@@
     (stroke (width 0) (type default))
   )
+  (wire (pts (xy 46.99 101.6) (xy 100.33 101.6))
+    (stroke (width 0) (type default))
+  )
   (wire (pts (xy 93.98 55.88) (xy 93.98 71.12))
     (stroke (width 0) (type default))
@@
     (stroke (width 0) (type default))
   )
-  (wire (pts (xy 35.56 99.06) (xy 110.49 99.06))
+  (wire (pts (xy 35.56 99.06) (xy 39.37 99.06))
     (stroke (width 0) (type default))
   )
@@
     )
   )
+  (text "√" (at 26.67 100.33 0)
+    (effects (font (size 1.27 1.27)) (justify left bottom))
+  )
   (text "Keypad" (at 27.94 17.78 0)
     (effects (font (size 1.27 1.27)) (justify left bottom))
@@
     (effects (font (size 1.27 1.27)) (justify left bottom))
   )
+  (text "√" (at 26.67 97.79 0)
+    (effects (font (size 1.27 1.27)) (justify left bottom))
+  )
   (text "Backlight" (at 220.98 20.32 0)
     (effects (font (size 1.27 1.27)) (justify left bottom))
@@
     )
   )
+  (symbol (lib_id "UV-K5:R") (at 43.18 93.98 90) (unit 1)
+    (in_bom yes) (on_board yes) (dnp no)
+    (property "Reference" "R223" (at 49.53 92.71 90)
+      (effects (font (size 1.27 1.27)))
+    )
+    (property "Value" "1k" (at 43.18 93.98 90)
+      (effects (font (size 1.27 1.27)))
+    )
+    (property "Footprint" "" (at 43.18 95.758 90)
+      (effects (font (size 1.27 1.27)) hide)
+    )
+    (property "Datasheet" "~" (at 43.18 93.98 0)
+      (effects (font (size 1.27 1.27)) hide)
+    )
+    (pin "1")
+    (pin "2")
+    (instances
+      (project "UVK5_reversing"
+        (path "/abeb0e11-6961-4a93-ba06-0741c65258e1/5a511d47-c886-48a4-9f6d-e26c2c56ff6f"
+          (reference "R223") (unit 1)
+        )
+      )
+    )
+  )
   (symbol (lib_id "UV-K5:R") (at 69.85 118.11 180) (unit 1)
     (in_bom yes) (on_board yes) (dnp no) (fields_autoplaced)
@@
     )
   )
+  (symbol (lib_id "UV-K5:R") (at 43.18 99.06 90) (unit 1)
+    (in_bom yes) (on_board yes) (dnp no)
+    (property "Reference" "R193" (at 49.53 97.79 90)
+      (effects (font (size 1.27 1.27)))
+    )
+    (property "Value" "100R" (at 43.18 99.06 90)
+      (effects (font (size 1.27 1.27)))
+    )
+    (property "Footprint" "" (at 43.18 100.838 90)
+      (effects (font (size 1.27 1.27)) hide)
+    )
+    (property "Datasheet" "~" (at 43.18 99.06 0)
+      (effects (font (size 1.27 1.27)) hide)
+    )
+    (pin "1")
+    (pin "2")
+    (instances
+      (project "UVK5_reversing"
+        (path "/abeb0e11-6961-4a93-ba06-0741c65258e1/5a511d47-c886-48a4-9f6d-e26c2c56ff6f"
+          (reference "R193") (unit 1)
+        )
+      )
+    )
+  )
   (symbol (lib_id "UV-K5:SW_Push") (at 82.55 111.76 0) (unit 1)
     (in_bom yes) (on_board yes) (dnp no) (fields_autoplaced)
@@
     )
   )
+  (symbol (lib_id "UV-K5:R") (at 43.18 91.44 90) (unit 1)
+    (in_bom yes) (on_board yes) (dnp no)
+    (property "Reference" "R227" (at 49.53 90.17 90)
+      (effects (font (size 1.27 1.27)))
+    )
+    (property "Value" "1k" (at 43.18 91.44 90)
+      (effects (font (size 1.27 1.27)))
+    )
+    (property "Footprint" "" (at 43.18 93.218 90)
+      (effects (font (size 1.27 1.27)) hide)
+    )
+    (property "Datasheet" "~" (at 43.18 91.44 0)
+      (effects (font (size 1.27 1.27)) hide)
+    )
+    (pin "1")
+    (pin "2")
+    (instances
+      (project "UVK5_reversing"
+        (path "/abeb0e11-6961-4a93-ba06-0741c65258e1/5a511d47-c886-48a4-9f6d-e26c2c56ff6f"
+          (reference "R227") (unit 1)
+        )
+      )
+    )
+  )
   (symbol (lib_id "UV-K5:R") (at 87.63 118.11 180) (unit 1)
     (in_bom yes) (on_board yes) (dnp no) (fields_autoplaced)
@@
         )
       )
+    )
+  )
+  (symbol (lib_id "UV-K5:R") (at 43.18 96.52 90) (unit 1)
+    (in_bom yes) (on_board yes) (dnp no)
+    (property "Reference" "R206" (at 49.53 95.25 90)
+      (effects (font (size 1.27 1.27)))
+    )
+    (property "Value" "100R" (at 43.18 96.52 90)
+      (effects (font (size 1.27 1.27)))
+    )
+    (property "Footprint" "" (at 43.18 98.298 90)
+      (effects (font (size 1.27 1.27)) hide)
+    )
+    (property "Datasheet" "~" (at 43.18 96.52 0)
+      (effects (font (size 1.27 1.27)) hide)
+    )
+    (pin "1")
+    (pin "2")
+    (instances
+      (project "UVK5_reversing"
+        (path "/abeb0e11-6961-4a93-ba06-0741c65258e1/5a511d47-c886-48a4-9f6d-e26c2c56ff6f"
+          (reference "R206") (unit 1)
+        )
+      )
