File: hardware/KiCad/Kicad_UVK5_reversing20230909/UVK5_reversing.kicad_sch (KiCad schematic)
At the start: 0 parts

Commit message: Add files via upload
Other:
- sheet Audio renamed Audio LN4898
- added sheet FM_BK1080 (FM_BK1080.kicad_sch)
Changed lines of the file:
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@@
     (stroke (width 1) (type solid))
     (fill (color 0 0 0 0.0000))
-    (property "Sheetname" "Audio" (at 63.5 92.8446 0)
+    (property "Sheetname" "Audio LN4898" (at 63.5 92.8446 0)
       (effects (font (size 1.27 1.27)) (justify left bottom))
     )
@@
       )
     )
+  )
+  (sheet (at 63.5 72.39) (size 12.7 11.43) (fields_autoplaced)
+    (stroke (width 1) (type solid))
+    (fill (color 0 0 0 0.0000))
+    (property "Sheetname" "FM_BK1080" (at 63.5 71.6784 0)
+      (effects (font (size 1.27 1.27)) (justify left bottom))
+    )
+    (property "Sheetfile" "FM_BK1080.kicad_sch" (at 63.5 84.4046 0)
+      (effects (font (size 1.27 1.27)) (justify left top))
+    )
+    (instances
+      (project "UVK5_reversing"
+        (path "/abeb0e11-6961-4a93-ba06-0741c65258e1" (page "14"))
+      )
+    )
