File: hardware/KiCad/Kicad_UVK5_reversing20230909/FM_BK1080.kicad_sch (KiCad schematic)
At the start: 23 parts, among them Q03 DTC114E, Q25 NPN, U26 BK1080VB

Commit message: Add files via upload
Parts:
- renumbered R83 to R591, R80 to R592, R81 to R607, R82 to R608
Changed lines of the file:
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@@
   (symbol (lib_id "Device:R") (at 127 67.31 90) (unit 1)
     (in_bom yes) (on_board yes) (dnp no)
-    (property "Reference" "R82" (at 132.08 66.04 90)
+    (property "Reference" "R608" (at 132.08 66.04 90)
       (effects (font (size 1.27 1.27)))
     )
@@
       (project "UVK5_reversing"
         (path "/abeb0e11-6961-4a93-ba06-0741c65258e1/8249b2ea-40b3-4476-8cc6-5da6040bf04c"
-          (reference "R82") (unit 1)
+          (reference "R608") (unit 1)
         )
       )
@@
   (symbol (lib_id "Device:R") (at 127 64.77 90) (unit 1)
     (in_bom yes) (on_board yes) (dnp no)
-    (property "Reference" "R81" (at 132.08 63.5 90)
+    (property "Reference" "R607" (at 132.08 63.5 90)
       (effects (font (size 1.27 1.27)))
     )
@@
       (project "UVK5_reversing"
         (path "/abeb0e11-6961-4a93-ba06-0741c65258e1/8249b2ea-40b3-4476-8cc6-5da6040bf04c"
-          (reference "R81") (unit 1)
+          (reference "R607") (unit 1)
         )
       )
@@
   (symbol (lib_id "Device:R") (at 163.83 69.85 90) (unit 1)
     (in_bom yes) (on_board yes) (dnp no)
-    (property "Reference" "R83" (at 163.83 72.39 90)
+    (property "Reference" "R591" (at 163.83 72.39 90)
       (effects (font (size 1.27 1.27)))
     )
@@
       (project "UVK5_reversing"
         (path "/abeb0e11-6961-4a93-ba06-0741c65258e1/8249b2ea-40b3-4476-8cc6-5da6040bf04c"
-          (reference "R83") (unit 1)
+          (reference "R591") (unit 1)
         )
       )
@@
   (symbol (lib_id "Device:R") (at 163.83 64.77 90) (unit 1)
     (in_bom yes) (on_board yes) (dnp no)
-    (property "Reference" "R80" (at 163.83 62.23 90)
+    (property "Reference" "R592" (at 163.83 62.23 90)
       (effects (font (size 1.27 1.27)))
     )
@@
       (project "UVK5_reversing"
         (path "/abeb0e11-6961-4a93-ba06-0741c65258e1/8249b2ea-40b3-4476-8cc6-5da6040bf04c"
-          (reference "R80") (unit 1)
-        )
-      )
+          (reference "R592") (unit 1)
+        )
+      )
