File: hardware/KiCad/Kicad_UVK5_reversing20230909/Gabiz_ro.kicad_sch (KiCad schematic)
At the start: 66 parts, among them J37 Conn_Coaxial, Q08 24 NPN, Q23 24 NPN, Q9 R24 NPN, U3 C4_TLV70013_SOT23-5, U5 C4_TLV70013_SOT23-5, U6 C4_TLV70013_SOT23-5

Commit message: Add files via upload
Parts:
- C95: value C -> 1.10pF
- renumbered Q9 to Q09
Connections:
- net U9_PA0 renamed U7_GP00
- net U9_PA3 renamed U7_GP03
- net U9_PA4 renamed U7_GP04
Other:
- moved on the sheet: C128, C137, C163, C82, C83, D12, D18, D19, Q23, R129, R143

Commit message: Add files via upload
Parts:
- L112: value 0.01µH -> 68.6nH
- Q08: value 24 NPN -> R24 NPN
Connections:
- net BAND_X renamed BAND_VHF
- net BAND_Y renamed BAND_UHF
Changed lines of the file:
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@@
   (title_block
     (title "UV-K5 RX Input (Parts-List-Numbering)")
+    (date "2023-09-15")
     (rev "ludwich")
     (comment 2 "https://github.com/ludwich66/Quansheng_UV-K5_Wiki/wiki/Parts---Teile")
@@
     )
   )
-  (global_label "BAND_Y" (shape input) (at 269.24 57.15 0) (fields_autoplaced)
+  (global_label "BAND_UHF" (shape input) (at 269.24 57.15 0) (fields_autoplaced)
     (effects (font (size 1.27 1.27)) (justify left))
-    (property "Intersheetrefs" "${INTERSHEET_REFS}" (at 279.2405 57.15 0)
-      (effects (font (size 1.27 1.27)) (justify left))
-    )
-  )
-  (global_label "BAND_X" (shape input) (at 260.35 24.13 0) (fields_autoplaced)
+    (property "Intersheetrefs" "${INTERSHEET_REFS}" (at 281.9015 57.15 0)
+      (effects (font (size 1.27 1.27)) (justify left))
+    )
+  )
+  (global_label "BAND_VHF" (shape input) (at 260.35 24.13 0) (fields_autoplaced)
     (effects (font (size 1.27 1.27)) (justify left))
-    (property "Intersheetrefs" "${INTERSHEET_REFS}" (at 270.4714 24.13 0)
+    (property "Intersheetrefs" "${INTERSHEET_REFS}" (at 272.7696 24.13 0)
       (effects (font (size 1.27 1.27)) (justify left))
     )
@@
     )
   )
-  (global_label "BAND_X" (shape input) (at 181.61 76.2 0) (fields_autoplaced)
+  (global_label "BAND_VHF" (shape input) (at 181.61 76.2 0) (fields_autoplaced)
     (effects (font (size 1.27 1.27)) (justify left))
-    (property "Intersheetrefs" "${INTERSHEET_REFS}" (at 191.7314 76.2 0)
+    (property "Intersheetrefs" "${INTERSHEET_REFS}" (at 194.0296 76.2 0)
       (effects (font (size 1.27 1.27)) (justify left))
     )
@@
     )
   )
-  (global_label "BAND_Y" (shape input) (at 180.34 130.81 0) (fields_autoplaced)
+  (global_label "BAND_UHF" (shape input) (at 180.34 130.81 0) (fields_autoplaced)
     (effects (font (size 1.27 1.27)) (justify left))
-    (property "Intersheetrefs" "${INTERSHEET_REFS}" (at 190.3405 130.81 0)
+    (property "Intersheetrefs" "${INTERSHEET_REFS}" (at 193.0015 130.81 0)
       (effects (font (size 1.27 1.27)) (justify left))
     )
@@
       (effects (font (size 1.27 1.27)))
     )
-    (property "Value" "0.01µH" (at 104.14 91.44 90)
+    (property "Value" "68.6nH" (at 104.14 91.44 90)
       (effects (font (size 1.27 1.27)))
     )
@@
       (effects (font (size 1.27 1.27)) (justify left))
     )
-    (property "Value" "24 NPN" (at 83.82 158.75 0)
-      (effects (font (size 1.27 1.27)) (justify left))
-    )
+    (property "Value" "R24 NPN" (at 83.82 158.75 0)
+      (effects (font (size 1.27 1.27)) (justify left))
+    )

Commit message: Add files via upload
Parts:
- C107: value 56pF -> 22pF
- C137: value 110nF -> 850pF
- L16: value 0.20µH -> 56nH
Other:
- moved on the sheet: C10, C108
Changed lines of the file:
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@@
   (title_block
     (title "UV-K5 RX Input (Parts-List-Numbering)")
-    (date "2023-09-15")
+    (date "2023-09-17")
     (rev "ludwich")
     (comment 2 "https://github.com/ludwich66/Quansheng_UV-K5_Wiki/wiki/Parts---Teile")
@@
     (stroke (width 0) (type default))
   )
-  (wire (pts (xy 68.58 139.7) (xy 68.58 140.97))
+  (wire (pts (xy 67.31 139.7) (xy 67.31 140.97))
     (stroke (width 0) (type default))
   )
@@
     (stroke (width 0) (type default))
   )
-  (wire (pts (xy 68.58 85.09) (xy 68.58 86.36))
+  (wire (pts (xy 67.31 85.09) (xy 67.31 86.36))
     (stroke (width 0) (type default))
   )
@@
     (stroke (width 0) (type default))
   )
-  (wire (pts (xy 68.58 130.81) (xy 68.58 132.08))
+  (wire (pts (xy 67.31 130.81) (xy 67.31 132.08))
     (stroke (width 0) (type default))
   )
@@
     (stroke (width 0) (type default))
   )
-  (wire (pts (xy 81.28 130.81) (xy 68.58 130.81))
+  (wire (pts (xy 81.28 130.81) (xy 67.31 130.81))
     (stroke (width 0) (type default))
   )
@@
     (stroke (width 0) (type default))
   )
-  (wire (pts (xy 81.28 76.2) (xy 68.58 76.2))
+  (wire (pts (xy 81.28 76.2) (xy 67.31 76.2))
     (stroke (width 0) (type default))
   )
@@
     (stroke (width 0) (type default))
   )
-  (wire (pts (xy 68.58 76.2) (xy 68.58 77.47))
+  (wire (pts (xy 67.31 76.2) (xy 67.31 77.47))
     (stroke (width 0) (type default))
   )
@@
       (effects (font (size 1.27 1.27)))
     )
-    (property "Value" "110nF" (at 143.51 88.9 90)
+    (property "Value" "850pF" (at 143.51 88.9 90)
       (effects (font (size 1.27 1.27)))
     )
@@
     )
   )
-  (symbol (lib_id "power:GND") (at 68.58 140.97 0) (unit 1)
+  (symbol (lib_id "power:GND") (at 67.31 140.97 0) (unit 1)
     (in_bom yes) (on_board yes) (dnp no) (fields_autoplaced)
-    (property "Reference" "#PWR0137" (at 68.58 147.32 0)
+    (property "Reference" "#PWR0137" (at 67.31 147.32 0)
       (effects (font (size 1.27 1.27)) hide)
     )
-    (property "Value" "GND" (at 68.58 146.05 0)
+    (property "Value" "GND" (at 67.31 146.05 0)
       (effects (font (size 1.27 1.27)))
     )
-    (property "Footprint" "" (at 68.58 140.97 0)
+    (property "Footprint" "" (at 67.31 140.97 0)
       (effects (font (size 1.27 1.27)) hide)
     )
-    (property "Datasheet" "" (at 68.58 140.97 0)
+    (property "Datasheet" "" (at 67.31 140.97 0)
       (effects (font (size 1.27 1.27)) hide)
     )
@@
     )
   )
-  (symbol (lib_id "Device:C") (at 68.58 135.89 0) (unit 1)
+  (symbol (lib_id "Device:C") (at 67.31 135.89 0) (unit 1)
     (in_bom yes) (on_board yes) (dnp no) (fields_autoplaced)
-    (property "Reference" "C10" (at 72.39 134.62 0)
+    (property "Reference" "C10" (at 71.12 134.62 0)
       (effects (font (size 1.27 1.27)) (justify left))
     )
-    (property "Value" "10nF" (at 72.39 137.16 0)
+    (property "Value" "10nF" (at 71.12 137.16 0)
       (effects (font (size 1.27 1.27)) (justify left))
     )
-    (property "Footprint" "" (at 69.5452 139.7 0)
+    (property "Footprint" "" (at 68.2752 139.7 0)
       (effects (font (size 1.27 1.27)) hide)
     )
-    (property "Datasheet" "~" (at 68.58 135.89 0)
+    (property "Datasheet" "~" (at 67.31 135.89 0)
       (effects (font (size 1.27 1.27)) hide)
     )
@@
       (effects (font (size 1.27 1.27)))
     )
-    (property "Value" "56pF" (at 92.71 88.9 90)
+    (property "Value" "22pF" (at 92.71 88.9 90)
       (effects (font (size 1.27 1.27)))
     )
@@
       (effects (font (size 1.27 1.27)))
     )
-    (property "Value" "0.20µH" (at 34.29 100.33 90)
+    (property "Value" "56nH" (at 34.29 100.33 90)
       (effects (font (size 1.27 1.27)))
     )
@@
     )
   )
-  (symbol (lib_id "Device:C") (at 68.58 81.28 0) (unit 1)
+  (symbol (lib_id "Device:C") (at 67.31 81.28 0) (unit 1)
     (in_bom yes) (on_board yes) (dnp no) (fields_autoplaced)
-    (property "Reference" "C108" (at 72.39 80.01 0)
+    (property "Reference" "C108" (at 71.12 80.01 0)
       (effects (font (size 1.27 1.27)) (justify left))
     )
-    (property "Value" "10nF" (at 72.39 82.55 0)
+    (property "Value" "10nF" (at 71.12 82.55 0)
       (effects (font (size 1.27 1.27)) (justify left))
     )
-    (property "Footprint" "" (at 69.5452 85.09 0)
+    (property "Footprint" "" (at 68.2752 85.09 0)
       (effects (font (size 1.27 1.27)) hide)
     )
-    (property "Datasheet" "~" (at 68.58 81.28 0)
+    (property "Datasheet" "~" (at 67.31 81.28 0)
       (effects (font (size 1.27 1.27)) hide)
     )
@@
     )
   )
-  (symbol (lib_id "power:GND") (at 68.58 86.36 0) (unit 1)
+  (symbol (lib_id "power:GND") (at 67.31 86.36 0) (unit 1)
     (in_bom yes) (on_board yes) (dnp no) (fields_autoplaced)
-    (property "Reference" "#PWR0125" (at 68.58 92.71 0)
+    (property "Reference" "#PWR0125" (at 67.31 92.71 0)
       (effects (font (size 1.27 1.27)) hide)
     )
-    (property "Value" "GND" (at 68.58 91.44 0)
+    (property "Value" "GND" (at 67.31 91.44 0)
       (effects (font (size 1.27 1.27)))
     )
-    (property "Footprint" "" (at 68.58 86.36 0)
+    (property "Footprint" "" (at 67.31 86.36 0)
       (effects (font (size 1.27 1.27)) hide)
     )
-    (property "Datasheet" "" (at 68.58 86.36 0)
+    (property "Datasheet" "" (at 67.31 86.36 0)
       (effects (font (size 1.27 1.27)) hide)
     )
